File: bobbycar-lora-can-ethernet.kicad_sch (KiCad schematic)
At the start: 64 parts, among them J1 Conn_01x04, J2 Conn_01x04, J3 ATGM336H-5N31, J4 Micro_SD_Card_Det_Hirose_DM3AT, J5 Wuerth_7499010121A, Q1 SS8050_C2150, Q2 SS8050_C2150, U1 ESP32-WROOM-32E, U2 Ai-Thinker-Ra-01SH, U3 LM75B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

Commit message: improve README, add component number in schematics
Parts:
- D3: symbol Device:D -> Device:D_Schottky
- U7: value MPM2359 -> TPMP2359DJ
Changed lines of the file:
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@@
     (pin "1")
   )
-  (symbol (lib_id "Device:D") (at 264.16 34.29 270) (unit 1)
+  (symbol (lib_id "Device:D_Schottky") (at 264.16 34.29 270) (unit 1)
     (in_bom yes) (on_board yes) (fields_autoplaced)
     (property "Reference" "D3" (id 0) (at 266.192 33.3815 90)
@@
     (in_bom yes) (on_board yes)
     (property "Reference" "U7" (id 0) (at 353.06 66.929 0))
-    (property "Value" "MPM2359" (id 1) (at 353.06 69.2404 0))
+    (property "Value" "TPMP2359DJ" (id 1) (at 353.06 69.2404 0))
     (property "Footprint" "Package_TO_SOT_SMD:SOT-23-6" (id 2) (at 370.84 87.63 0)
       (effects (font (size 1.27 1.27)) hide)
@@
     )
     (path "/9e495491-eacb-47b2-9a0f-1360dcedc080"
-      (reference "U7") (unit 1) (value "MPM2359") (footprint "Package_TO_SOT_SMD:SOT-23-6")
+      (reference "U7") (unit 1) (value "TPMP2359DJ") (footprint "Package_TO_SOT_SMD:SOT-23-6")
     )
     (path "/41dcc8d5-1bb1-4742-95f6-344bfb8ddac7"
